File: blind pcb.kicad_pcb (KiCad board)
At the start: 2 copper layers, 73.8 x 59.3 mm, 27 parts, among them J1 Screw_Terminal_01x02, J2 Screw_Terminal_01x02, J3 Screw_Terminal_01x02, J4 Screw_Terminal_01x02, J5 Screw_Terminal_01x02, Q1 AO3400A, Q2 AO3400A, Q3 AO3400A, Q4 AO3400A, SW1 SW_SPDT

Commit message: clean up
Parts:
- Arduino Nano: renamed from A1
- Voltage Converter: renamed from 1
Routing:
- net Net-(A1-D3): track 30.7 -> 31.8 mm
- net Net-(A1-D8): track 53.8 -> 53.2 mm
Changed lines of the file:
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@@
 		(layer "F.Cu")
 		(at 158.025 98.525)
-		(property "Reference" "1"
-			(at 3 1 0)
+		(property "Reference" "Voltage Converter"
+			(at -1.025 -2.275 90)
 			(unlocked yes)
 			(layer "F.SilkS")
@@
 		(descr "Arduino Nano, http://www.mouser.com/pdfdocs/Gravitech_Arduino_Nano3_0.pdf")
 		(tags "Arduino Nano")
-		(property "Reference" "A1"
-			(at 13.96458 -8.975 270)
+		(property "Reference" "Arduino Nano"
+			(at 7.98958 -17.75 270)
 			(layer "B.SilkS")
 			(effects
@@
 	)
 	(segment
-		(start 159 105)
-		(end 154.8 109.2)
+		(start 161.2 92.8)
+		(end 161.2 95.675)
 		(width 0.254)
 		(layer "F.Cu")
@@
 	)
 	(segment
-		(start 161.007 94.803)
-		(end 161.007 96.75)
+		(start 159 105)
+		(end 154.8 109.2)
 		(width 0.254)
 		(layer "F.Cu")
@@
 	)
 	(segment
-		(start 161.007 96.75)
-		(end 159 98.757)
+		(start 159 97.875)
+		(end 159 105)
+		(width 0.254)
+		(layer "F.Cu")
+		(net "Net-(A1-D3)")
+	)
+	(segment
+		(start 168 86)
+		(end 161.2 92.8)
 		(width 0.254)
 		(layer "F.Cu")
@@
 	(segment
 		(start 169.81 86)
-		(end 161.007 94.803)
+		(end 168 86)
 		(width 0.254)
 		(layer "F.Cu")
@@
 	)
 	(segment
-		(start 159 98.757)
-		(end 159 105)
+		(start 161.2 95.675)
+		(end 159 97.875)
 		(width 0.254)
 		(layer "F.Cu")
@@
 	)
 	(segment
-		(start 171.219729 121.762329)
-		(end 171.219729 111.969729)
+		(start 171.219729 111.719729)
+		(end 168.454 108.954)
 		(width 0.254)
 		(layer "F.Cu")
@@
 	)
 	(segment
-		(start 171.219729 111.969729)
-		(end 168.204 108.954)
+		(start 171.219729 121.762329)
+		(end 171.219729 111.719729)
 		(width 0.254)
 		(layer "F.Cu")
@@
 	)
 	(segment
-		(start 168.204 108.954)
+		(start 168.454 108.954)
 		(end 158.87558 108.954)
 		(width 0.254)
@@
 	)
 	(segment
-		(start 172.439458 116.924087)
-		(end 167.131951 111.61658)
+		(start 167.265371 111.75)
+		(end 153.52042 111.75)
 		(width 0.254)
 		(layer "B.Cu")
@@
 	)
 	(segment
-		(start 153.387 111.61658)
-		(end 152.26 110.48958)
+		(start 172.439458 116.924087)
+		(end 167.265371 111.75)
 		(width 0.254)
 		(layer "B.Cu")
@@
 	)
 	(segment
-		(start 167.131951 111.61658)
-		(end 153.387 111.61658)
+		(start 153.52042 111.75)
+		(end 152.26 110.48958)
 		(width 0.254)
 		(layer "B.Cu")
@@
 	)
 	(segment
-		(start 140.75 96.75)
-		(end 149.72 105.72)
+		(start 132.897574 85.240414)
+		(end 140.8 93.14284)
 		(width 0.254)
 		(layer "B.Cu")
@@
 	)
 	(segment
-		(start 140.75 93.09284)
-		(end 140.75 96.75)
+		(start 140.8 96.8)
+		(end 149.72 105.72)
 		(width 0.254)
 		(layer "B.Cu")
@@
 	)
 	(segment
-		(start 132.897574 85.240414)
-		(end 140.75 93.09284)
+		(start 140.8 93.14284)
+		(end 140.8 96.8)
 		(width 0.254)
 		(layer "B.Cu")
@@
 	)
 	(segment
+		(start 172.280271 80.117663)
+		(end 172.280271 80.969729)
+		(width 0.254)
+		(layer "F.Cu")
+		(net "Net-(A1-D7)")
+	)
+	(segment
+		(start 172.280271 80.969729)
+		(end 158.6 94.65)
+		(width 0.254)
+		(layer "F.Cu")
+		(net "Net-(A1-D7)")
+	)
+	(segment
 		(start 154.5 108.75)
 		(end 146.5 108.75)
@@
 	)
 	(segment
-		(start 172.280271 80.969729)
-		(end 158.5 94.75)
+		(start 158.546 104.704)
+		(end 154.5 108.75)
 		(width 0.254)
 		(layer "F.Cu")
@@
 	)
 	(segment
-		(start 172.280271 80.117663)
-		(end 172.280271 80.969729)
+		(start 158.6 94.65)
+		(end 158.6 97.632948)
 		(width 0.254)
 		(layer "F.Cu")
@@
 	)
 	(segment
-		(start 158.5 94.75)
-		(end 158.5 104.75)
+		(start 158.6 97.632948)
+		(end 158.546 97.686948)
 		(width 0.254)
 		(layer "F.Cu")
@@
 	)
 	(segment
-		(start 158.5 104.75)
-		(end 154.5 108.75)
+		(start 158.546 97.686948)
+		(end 158.546 104.704)
 		(width 0.254)
 		(layer "F.Cu")
@@
 	)
 	(segment
-		(start 156 96.75)
-		(end 158.046 98.796)
+		(start 156.75 94)
+		(end 156 94.75)
 		(width 0.254)
 		(layer "F.Cu")
@@
 	)
 	(segment
-		(start 143.33958 109.25)
-		(end 142.1 110.48958)
+		(start 154.357948 108.25)
+		(end 146.25 108.25)
 		(width 0.254)
 		(layer "F.Cu")
@@
 	)
 	(segment
-		(start 158.046 104.561948)
-		(end 154.357948 108.25)
+		(start 156 94.75)
+		(end 156 95.75)
 		(width 0.254)
 		(layer "F.Cu")
@@
 	)
 	(segment
-		(start 154.357948 108.25)
-		(end 146.25 108.25)
+		(start 171.060542 81.547406)
+		(end 158.607948 94)
 		(width 0.254)
 		(layer "F.Cu")
@@
 	)
 	(segment
-		(start 171.060542 81.547406)
-		(end 159.607948 93)
+		(start 145.25 109.25)
+		(end 143.33958 109.25)
 		(width 0.254)
 		(layer "F.Cu")
@@
 	)
 	(segment
-		(start 156 93.75)
-		(end 156 96.75)
+		(start 156 95.75)
+		(end 158.046 97.796)
 		(width 0.254)
 		(layer "F.Cu")
@@
 	)
 	(segment
-		(start 145.25 109.25)
-		(end 143.33958 109.25)
+		(start 158.607948 94)
+		(end 156.75 94)
 		(width 0.254)
 		(layer "F.Cu")
@@
 	)
 	(segment
-		(start 159.607948 93)
-		(end 156.75 93)
+		(start 146.25 108.25)
+		(end 145.25 109.25)
 		(width 0.254)
 		(layer "F.Cu")
@@
 	)
 	(segment
-		(start 156.75 93)
-		(end 156 93.75)
+		(start 143.33958 109.25)
+		(end 142.1 110.48958)
 		(width 0.254)
 		(layer "F.Cu")
@@
 	)
 	(segment
-		(start 158.046 98.796)
-		(end 158.046 104.561948)
+		(start 158.046 104.561948)
+		(end 154.357948 108.25)
 		(width 0.254)
 		(layer "F.Cu")
@@
 	)
 	(segment
-		(start 146.25 108.25)
-		(end 145.25 109.25)
+		(start 158.046 97.796)
+		(end 158.046 104.561948)
 		(width 0.254)
 		(layer "F.Cu")
