File: blind pcb.kicad_pcb (KiCad board)
At the start: 2 copper layers, 73.8 x 59.3 mm, 27 parts, among them J1 Screw_Terminal_01x02, J2 Screw_Terminal_01x02, J3 Screw_Terminal_01x02, J4 Screw_Terminal_01x02, J5 Screw_Terminal_01x02, Q1 AO3400A, Q2 AO3400A, Q3 AO3400A, Q4 AO3400A, SW1 SW_SPDT

Commit message: reroute
Parts:
- added R5: 10kΩ, Resistor_THT:R_Axial_DIN0207_L6.3mm_D2.5mm_P7.62mm_Horizontal, F.Cu at (176.8, 106.2)
- added R6: 10kΩ, Resistor_THT:R_Axial_DIN0207_L6.3mm_D2.5mm_P7.62mm_Horizontal, F.Cu at (124.7, 113.0)
- added R7: 10kΩ, Resistor_THT:R_Axial_DIN0207_L6.3mm_D2.5mm_P7.62mm_Horizontal, F.Cu at (128.2, 89.5)
- added R8: 10kΩ, Resistor_THT:R_Axial_DIN0207_L6.3mm_D2.5mm_P7.62mm_Horizontal, F.Cu at (175.5, 95.8)
- moved Arduino_Nano1 0.12 mm to (167.4, 110.4)
- renumbered A1 to Arduino_Nano1, 1 to MT3608
Connections:
- Arduino_Nano1 pad 5: Net-(A1-D2) -> Net-(Arduino_Nano1-D2)
- Arduino_Nano1 pad 6: unconnected-(A1-D3-Pad6) -> Net-(Arduino_Nano1-D3)
- Arduino_Nano1 pad 8: Net-(A1-D5) -> unconnected-(Arduino_Nano1-D5-Pad8)
- R4 pad 2: Net-(A1-D5) -> Net-(Arduino_Nano1-D2)
- S1 pad 2: Net-(A1-D2) -> Net-(Arduino_Nano1-D3)
Routing:
- net Net-(Arduino_Nano1-D3): track 0.00 -> 29.5 mm
- net Net-(A1-D2): track 26.0 -> 0.00 mm
- net Net-(A1-D5): track 22.3 -> 0.00 mm
- net Net-(Arduino_Nano1-D2): track 0.00 -> 20.6 mm
- net Net-(Q1-G): track 6.07 -> 17.5 mm
- net Net-(Q3-G): track 3.28 -> 12.7 mm
- net Net-(Q4-G): track 6.75 -> 15.3 mm
- net Net-(Q2-G): track 3.06 -> 8.52 mm
- net /5V: track 220.3 -> 225.0 mm
- net Net-(D2-A): track 19.0 -> 21.5 mm
- net Net-(MT3608-IN+): track 24.1 -> 25.4 mm
- net Net-(Arduino_Nano1-D4): track 30.1 -> 31.1 mm
- net Net-(Arduino_Nano1-A4): track 29.6 -> 30.5 mm
- net Net-(Arduino_Nano1-A3): track 33.5 -> 34.4 mm
- net /GND: track 0.00 -> 0.30 mm, vias 1 -> 0
Other:
- board text added: "+"
- board text added: "-"
- board text added: "100nF"
- board text added: "10kΩ"
- board text added: "220Ω"
- board text added: "IN+"
- board text added: "IN-"
- board text added: "JLCJLCJLCJLC"
- board text added: "OFF"
- board text added: "ON"
- board text added: "OUT+"
- board text added: "OUT-"
- board text added: "VCC"
