File: blind pcb.kicad_sch (KiCad schematic)
At the start: 27 parts, among them J1 Screw_Terminal_01x02, J2 Screw_Terminal_01x02, J3 Screw_Terminal_01x02, J4 Screw_Terminal_01x02, J5 Screw_Terminal_01x02, Q1 AO3400A, Q2 AO3400A, Q3 AO3400A, Q4 AO3400A, SW1 SW_SPDT

Commit message: reroute with ground plane
Connections:
- net 5V: now reaches 1.3 (OUT+), A1.27 (+5V), C1.1, C2.1, C3.1, C4.1, C5.1, D1.1 (K), D2.1 (K), D3.1 (K), D4.1 (K), J1.2 (Pin_2), J2.2 (Pin_2), J3.2 (Pin_2), J4.2 (Pin_2), S1.1 (Pin_1), S2.1 (Pin_1)
- net at R4.2: now also A1.8 (D5); no longer A1.12 (D9)
- net GND: now reaches 1.4 (OUT-), A1.29 (GND), A1.4 (GND), C1.2, Q1.2 (S), Q2.2 (S), Q3.2 (S), Q4.2 (S), S1.4 (Pin_4), S2.4 (Pin_4)
- net GND: now also 1.1 (IN-), J5.1 (Pin_1)
- net at S2.2 (Pin_2): now also A1.23 (A4); no longer A1.10 (D7)
- net at S2.3 (Pin_3): now also A1.22 (A3); no longer A1.11 (D8)
- net at A1.21 (A2): now also R2.2
- net at A1.24 (A5): now also R1.2
- net at A1.6 (D3): no longer R1.2

Commit message: reroute
Parts:
- added R5, R6, R7, R8: 10kΩ, Resistor_THT:R_Axial_DIN0207_L6.3mm_D2.5mm_P7.62mm_Horizontal, symbol Device:R
- renumbered A1 to Arduino_Nano1, 1 to MT3608
Connections:
- net GND: now also R5.1, R6.1, R7.1, R8.1
- net at Q4.1 (G), R4.1: now also R5.2
- net at R4.2: now also Arduino_Nano1.5 (D2); no longer Arduino_Nano1.8 (D5)
- net at Q3.1 (G), R3.1: now also R6.2
- net at Q2.1 (G), R2.1: now also R7.2
- net at Q1.1 (G), R1.1: now also R8.2
- net at S1.2 (Pin_2): now also Arduino_Nano1.6 (D3); no longer Arduino_Nano1.5 (D2)
